File: pcb-esp32-power.sch (KiCad schematic (older format))
At the start: 16 parts, among them IC2 SY8008B, J1 DB9_Female, J2 Conn_01x02, J3 Conn_01x14, J4 Conn_01x16, U1 STEPDOWN12_5

Commit message: ESP32 Bus verwendet
Parts:
- removed J3: Conn_01x14, Connector_PinSocket_2.54mm:PinSocket_1x14_P2.54mm_Vertical, symbol Connector_Generic:Conn_01x14
- removed J4: Conn_01x16, Connector_PinSocket_2.54mm:PinSocket_1x16_P2.54mm_Vertical, symbol Connector_Generic:Conn_01x16
- added J3: Bus_Connector, esp32bus:PinHeader, symbol ESP32_Bus:Bus_Connector
Connections:
- wire segments 55 -> 65
- no-connect marks 4 -> 25
Changed lines of the file:
@@
-	1    0    0    -1
-$EndComp
-$Comp
-L Connector_Generic:Conn_01x16 J4
-U 1 1 60DF91CB
-P 7700 1650
-F 0 "J4" H 7780 1692 50  0000 L CNN
-F 1 "Conn_01x16" H 7780 1601 50  0000 L CNN
-F 2 "Connector_PinSocket_2.54mm:PinSocket_1x16_P2.54mm_Vertical" H 7700 1650 50  0001 C CNN
-F 3 "~" H 7700 1650 50  0001 C CNN
-	1    7700 1650
-	1    0    0    -1
-$EndComp
-$Comp
-L Connector_Generic:Conn_01x14 J3
-U 1 1 60DF886D
-P 6100 1650
-F 0 "J3" H 6180 1692 50  0000 L CNN
-F 1 "Conn_01x14" H 6180 1601 50  0000 L CNN
-F 2 "Connector_PinSocket_2.54mm:PinSocket_1x14_P2.54mm_Vertical" H 6100 1650 50  0001 C CNN
-F 3 "~" H 6100 1650 50  0001 C CNN
-	1    6100 1650
 	1    0    0    -1
 $EndComp
@@
 	1    0    0    -1
 $EndComp
-Text GLabel 5900 1550 0    50   Input ~ 0
+Text GLabel 2500 4000 0    50   Input ~ 0
 EXTPOW
-Text GLabel 7500 1450 0    50   Input ~ 0
+Text GLabel 3700 4000 2    50   Input ~ 0
 SDA
-Text GLabel 7500 1150 0    50   Input ~ 0
+Text GLabel 3700 3700 2    50   Input ~ 0
 SCL
-Text GLabel 5900 2050 0    50   Input ~ 0
+Text GLabel 2500 4500 0    50   Input ~ 0
 INT
+$Comp
+L ESP32_Bus:Bus_Connector J3
+U 1 1 60F7276E
+P 3100 3850
+F 0 "J3" H 3100 4593 60  0000 C CNN
+F 1 "Bus_Connector" H 3100 4487 60  0000 C CNN
+F 2 "esp32bus:PinHeader" H 3100 4381 60  0000 C CNN
+F 3 "" H 3650 3150 60  0000 C CNN
+	1    3100 3850
+	1    0    0    -1
+$EndComp
+Wire Wire Line
+	2500 4000 2600 4000
+Wire Wire Line
+	2500 4500 2600 4500
+Wire Wire Line
+	3600 3700 3700 3700
+Wire Wire Line
+	3600 4000 3700 4000
+$Comp
+L power:GND #PWR0121
+U 1 1 60F7A061
+P 3700 3400
+F 0 "#PWR0121" H 3700 3150 50  0001 C CNN
+F 1 "GND" H 3705 3227 50  0000 C CNN
+F 2 "" H 3700 3400 50  0001 C CNN
+F 3 "" H 3700 3400 50  0001 C CNN
+	1    3700 3400
+	-1   0    0    1
+$EndComp
+Wire Wire Line
+	3600 3500 3700 3500
+Wire Wire Line
+	3700 3500 3700 3400
+$Comp
+L power:+3.3V #PWR0122
+U 1 1 60F7BA28
+P 2450 3400
+F 0 "#PWR0122" H 2450 3250 50  0001 C CNN
+F 1 "+3.3V" H 2465 3573 50  0000 C CNN
+F 2 "" H 2450 3400 50  0001 C CNN
+F 3 "" H 2450 3400 50  0001 C CNN
+	1    2450 3400
+	1    0    0    -1
+$EndComp
+Wire Wire Line
+	2450 3400 2450 3500
+Wire Wire Line
+	2450 3500 2600 3500
+NoConn ~ 2600 3600
+NoConn ~ 2600 3700
+NoConn ~ 2600 3800
+NoConn ~ 2600 3900
+NoConn ~ 2600 4100
+NoConn ~ 2600 4200
+NoConn ~ 2600 4300
+NoConn ~ 2600 4400
+NoConn ~ 2600 4600
+NoConn ~ 2600 4700
+NoConn ~ 2600 4800
+NoConn ~ 3600 3600
+NoConn ~ 3600 3800
+NoConn ~ 3600 3900
+NoConn ~ 3600 4100
+NoConn ~ 3600 4200
+NoConn ~ 3600 4300
+NoConn ~ 3600 4400
+NoConn ~ 3600 4500
+NoConn ~ 3600 4600
+NoConn ~ 3600 4700
+Text GLabel 3700 5000 2    50   Input ~ 0
+CANH
+Text GLabel 3700 4900 2    50   Input ~ 0
+CANL
+Wire Wire Line
+	3600 4900 3700 4900
+Wire Wire Line
+	3600 5000 3700 5000
 $EndSCHEMATC

Commit message: Mit OBD II Stecker
Parts:
- removed J1: DB9_Female, Connector_Dsub:DSUB-9_Female_Horizontal_P2.77x2.84mm_EdgePinOffset4.94mm_Housed_MountingHolesOffset7.48mm, symbol Connector:DB9_Female
- added J1: C-OBD-II-16M, OBD-II:COMTECH_C-OBD-II-16M, symbol C-OBD-II-16M:C-OBD-II-16M
Connections:
- wire segments 65 -> 63
- no-connect marks 25 -> 33
Other:
- moved on the sheet: R6, R7, U1
Changed lines of the file:
@@
 $EndDescr
-$Comp
-L Connector:DB9_Female J1
-U 1 1 60D5B7BC
-P 950 1750
-F 0 "J1" H 868 1058 50  0000 C CNN
-F 1 "DB9_Female" H 868 1149 50  0000 C CNN
-F 2 "Connector_Dsub:DSUB-9_Female_Horizontal_P2.77x2.84mm_EdgePinOffset4.94mm_Housed_MountingHolesOffset7.48mm" H 950 1750 50  0001 C CNN
-F 3 " ~" H 950 1750 50  0001 C CNN
-	1    950  1750
-	-1   0    0    1
-$EndComp
-$Comp
-L power:+12V #PWR0106
-U 1 1 60D60D1E
-P 1550 1450
-F 0 "#PWR0106" H 1550 1300 50  0001 C CNN
-F 1 "+12V" H 1565 1623 50  0000 C CNN
-F 2 "" H 1550 1450 50  0001 C CNN
-F 3 "" H 1550 1450 50  0001 C CNN
-	1    1550 1450
-	1    0    0    -1
-$EndComp
-$Comp
-L power:GND #PWR0107
-U 1 1 60D61B83
-P 1550 2050
-F 0 "#PWR0107" H 1550 1800 50  0001 C CNN
-F 1 "GND" H 1555 1877 50  0000 C CNN
-F 2 "" H 1550 2050 50  0001 C CNN
-F 3 "" H 1550 2050 50  0001 C CNN
-	1    1550 2050
-	1    0    0    -1
-$EndComp
-Wire Wire Line
-	1250 1450 1550 1450
-Wire Wire Line
-	1250 1750 1550 1750
-Wire Wire Line
-	1550 1750 1550 2050
-Wire Wire Line
-	1250 2050 1550 2050
-Connection ~ 1550 2050
-NoConn ~ 1250 1350
-NoConn ~ 1250 1550
-NoConn ~ 1250 1650
-NoConn ~ 1250 2150
-Text GLabel 1700 1850 2    50   Input ~ 0
-CANH
-Text GLabel 1700 1950 2    50   Input ~ 0
-CANL
-Wire Wire Line
-	1250 1850 1700 1850
-Wire Wire Line
-	1250 1950 1700 1950
 $Comp
 L power:+12V #PWR0108
 U 1 1 60DA8AE4
-P 2400 1550
-F 0 "#PWR0108" H 2400 1400 50  0001 C CNN
-F 1 "+12V" H 2415 1723 50  0000 C CNN
-F 2 "" H 2400 1550 50  0001 C CNN
-F 3 "" H 2400 1550 50  0001 C CNN
-	1    2400 1550
+P 3350 1400
+F 0 "#PWR0108" H 3350 1250 50  0001 C CNN
+F 1 "+12V" H 3365 1573 50  0000 C CNN
+F 2 "" H 3350 1400 50  0001 C CNN
+F 3 "" H 3350 1400 50  0001 C CNN
+	1    3350 1400
 	1    0    0    -1
 $EndComp
@@
 L power:GND #PWR0109
 U 1 1 60DA924D
-P 2400 1850
-F 0 "#PWR0109" H 2400 1600 50  0001 C CNN
-F 1 "GND" H 2405 1677 50  0000 C CNN
-F 2 "" H 2400 1850 50  0001 C CNN
-F 3 "" H 2400 1850 50  0001 C CNN
-	1    2400 1850
-	1    0    0    -1
-$EndComp
-Wire Wire Line
-	2400 1550 2400 1650
-Wire Wire Line
-	2400 1650 2550 1650
-Wire Wire Line
-	2400 1850 2400 1750
-Wire Wire Line
-	2400 1750 2550 1750
-Wire Wire Line
-	2550 1550 2400 1550
-Connection ~ 2400 1550
-Wire Wire Line
-	2550 1850 2400 1850
-Connection ~ 2400 1850
-Text GLabel 3450 1550 2    50   Input ~ 0
+P 3350 1700
+F 0 "#PWR0109" H 3350 1450 50  0001 C CNN
+F 1 "GND" H 3355 1527 50  0000 C CNN
+F 2 "" H 3350 1700 50  0001 C CNN
+F 3 "" H 3350 1700 50  0001 C CNN
+	1    3350 1700
+	1    0    0    -1
+$EndComp
+Wire Wire Line
+	3350 1400 3350 1500
+Wire Wire Line
+	3350 1500 3500 1500
+Wire Wire Line
+	3350 1700 3350 1600
+Wire Wire Line
+	3350 1600 3500 1600
+Wire Wire Line
+	3500 1400 3350 1400
+Connection ~ 3350 1400
+Wire Wire Line
+	3500 1700 3350 1700
+Connection ~ 3350 1700
+Text GLabel 4400 1400 2    50   Input ~ 0
 5VIN
 $Comp
 L power:GND #PWR0110
 U 1 1 60DB30D1
-P 3450 1850
-F 0 "#PWR0110" H 3450 1600 50  0001 C CNN
-F 1 "GND" H 3455 1677 50  0000 C CNN
-F 2 "" H 3450 1850 50  0001 C CNN
-F 3 "" H 3450 1850 50  0001 C CNN
-	1    3450 1850
-	1    0    0    -1
-$EndComp
-Wire Wire Line
-	3300 1650 3450 1650
-Wire Wire Line
-	3450 1650 3450 1550
-Wire Wire Line
-	3300 1550 3450 1550
-Wire Wire Line
-	3300 1750 3450 1750
-Wire Wire Line
-	3450 1750 3450 1850
-Wire Wire Line
-	3300 1850 3450 1850
-Connection ~ 3450 1850
+P 4400 1700
+F 0 "#PWR0110" H 4400 1450 50  0001 C CNN
+F 1 "GND" H 4405 1527 50  0000 C CNN
+F 2 "" H 4400 1700 50  0001 C CNN
+F 3 "" H 4400 1700 50  0001 C CNN
+	1    4400 1700
+	1    0    0    -1
+$EndComp
+Wire Wire Line
+	4250 1500 4400 1500
+Wire Wire Line
+	4400 1500 4400 1400
+Wire Wire Line
+	4250 1400 4400 1400
+Wire Wire Line
+	4250 1600 4400 1600
+Wire Wire Line
+	4400 1600 4400 1700
+Wire Wire Line
+	4250 1700 4400 1700
+Connection ~ 4400 1700
 $Comp
 L power:PWR_FLAG #FLG0101
@@
 L stepdown12_5:STEPDOWN12_5 U1
 U 1 1 60F48B5B
-P 2900 1950
-F 0 "U1" H 2875 1335 50  0000 C CNN
-F 1 "STEPDOWN12_5" H 2875 1426 50  0000 C CNN
-F 2 "StepDownBreakout:StepDownBreakout" H 2900 1950 50  0001 C CNN
-F 3 "" H 2900 1950 50  0001 C CNN
-	1    2900 1950
+P 3850 1800
+F 0 "U1" H 3825 1185 50  0000 C CNN
+F 1 "STEPDOWN12_5" H 3825 1276 50  0000 C CNN
+F 2 "StepDownBreakout:StepDownBreakout" H 3850 1800 50  0001 C CNN
+F 3 "" H 3850 1800 50  0001 C CNN
+	1    3850 1800
 	-1   0    0    1
 $EndComp
-Text GLabel 4400 1550 0    50   Input ~ 0
+Text GLabel 5350 1400 0    50   Input ~ 0
 5VIN
 $Comp
 L Device:R R6
 U 1 1 60F6141D
-P 4600 1700
-F 0 "R6" H 4670 1746 50  0000 L CNN
-F 1 "R" H 4670 1655 50  0000 L CNN
-F 2 "Resistor_SMD:R_0603_1608Metric" V 4530 1700 50  0001 C CNN
-F 3 "~" H 4600 1700 50  0001 C CNN
-	1    4600 1700
+P 5550 1550
+F 0 "R6" H 5620 1596 50  0000 L CNN
+F 1 "R" H 5620 1505 50  0000 L CNN
+F 2 "Resistor_SMD:R_0603_1608Metric" V 5480 1550 50  0001 C CNN
+F 3 "~" H 5550 1550 50  0001 C CNN
+	1    5550 1550
 	1    0    0    -1
 $EndComp
@@
 L Device:R R7
 U 1 1 60F61A44
-P 4600 2100
-F 0 "R7" H 4670 2146 50  0000 L CNN
-F 1 "R" H 4670 2055 50  0000 L CNN
-F 2 "Resistor_SMD:R_0603_1608Metric" V 4530 2100 50  0001 C CNN
-F 3 "~" H 4600 2100 50  0001 C CNN
-	1    4600 2100
-	1    0    0    -1
-$EndComp
-Text GLabel 4800 1900 2    50   Input ~ 0
+P 5550 1950
+F 0 "R7" H 5620 1996 50  0000 L CNN
+F 1 "R" H 5620 1905 50  0000 L CNN
+F 2 "Resistor_SMD:R_0603_1608Metric" V 5480 1950 50  0001 C CNN
+F 3 "~" H 5550 1950 50  0001 C CNN
+	1    5550 1950
+	1    0    0    -1
+$EndComp
+Text GLabel 5750 1750 2    50   Input ~ 0
 EXTPOW
 Wire Wire Line
-	4400 1550 4600 1550
-Wire Wire Line
-	4600 1850 4600 1900
-Wire Wire Line
-	4600 1900 4800 1900
-Connection ~ 4600 1900
-Wire Wire Line
-	4600 1900 4600 1950
+	5350 1400 5550 1400
+Wire Wire Line
+	5550 1700 5550 1750
+Wire Wire Line
+	5550 1750 5750 1750
+Connection ~ 5550 1750
+Wire Wire Line
+	5550 1750 5550 1800
 $Comp
 L power:GND #PWR0120
 U 1 1 60F64C82
-P 4600 2250
-F 0 "#PWR0120" H 4600 2000 50  0001 C CNN
-F 1 "GND" H 4605 2077 50  0000 C CNN
-F 2 "" H 4600 2250 50  0001 C CNN
-F 3 "" H 4600 2250 50  0001 C CNN
-	1    4600 2250
+P 5550 2100
+F 0 "#PWR0120" H 5550 1850 50  0001 C CNN
+F 1 "GND" H 5555 1927 50  0000 C CNN
+F 2 "" H 5550 2100 50  0001 C CNN
+F 3 "" H 5550 2100 50  0001 C CNN
+	1    5550 2100
 	1    0    0    -1
 $EndComp
@@
 Wire Wire Line
 	3600 5000 3700 5000
+$Comp
+L C-OBD-II-16M:C-OBD-II-16M J1
+U 1 1 6103A977
+P 1750 1500
+F 0 "J1" H 1750 2067 50  0000 C CNN
+F 1 "C-OBD-II-16M" H 1750 1976 50  0000 C CNN
+F 2 "OBD-II:COMTECH_C-OBD-II-16M" H 1750 1500 50  0001 L BNN
+F 3 "" H 1750 1500 50  0001 L BNN
+F 4 "Comtech Electronic Co." H 1750 1500 50  0001 L BNN "MANUFACTURER"
+F 5 "A" H 1750 1500 50  0001 L BNN "PARTREV"
+F 6 "Manufacturer Recommendations" H 1750 1500 50  0001 L BNN "STANDARD"
+F 7 "18.3mm" H 1750 1500 50  0001 L BNN "MAXIMUM_PACKAGE_HEIGHT"
+	1    1750 1500
+	1    0    0    -1
+$EndComp
+$Comp
+L power:+12V #PWR0106
+U 1 1 6103B5E2
+P 2400 1900
+F 0 "#PWR0106" H 2400 1750 50  0001 C CNN
+F 1 "+12V" H 2415 2073 50  0000 C CNN
+F 2 "" H 2400 1900 50  0001 C CNN
+F 3 "" H 2400 1900 50  0001 C CNN
+	1    2400 1900
+	-1   0    0    1
+$EndComp
+Text GLabel 1100 1700 0    50   Input ~ 0
+CANH
+Text GLabel 2400 1700 2    50   Input ~ 0
+CANL
+$Comp
+L power:GND #PWR0107
+U 1 1 6103C4CA
+P 1100 1600
+F 0 "#PWR0107" H 1100 1350 50  0001 C CNN
+F 1 "GND" H 1105 1427 50  0000 C CNN
+F 2 "" H 1100 1600 50  0001 C CNN
+F 3 "" H 1100 1600 50  0001 C CNN
+	1    1100 1600
+	-1   0    0    1
+$EndComp
+Wire Wire Line
+	1100 1600 1250 1600
+Wire Wire Line
+	1100 1700 1250 1700
+Wire Wire Line
+	2250 1700 2400 1700
+Wire Wire Line
+	2250 1900 2400 1900
+NoConn ~ 1250 1200
+NoConn ~ 1250 1300
+NoConn ~ 1250 1400
+NoConn ~ 1250 1500
+NoConn ~ 1250 1800
+NoConn ~ 1250 1900
+NoConn ~ 2250 1800
+NoConn ~ 2250 1600
+NoConn ~ 2250 1500
+NoConn ~ 2250 1400
+NoConn ~ 2250 1300
+NoConn ~ 2250 1200
 $EndSCHEMATC

Commit message: Footprints für "Hand solder"
Parts:
- C6: footprint Capacitor_SMD:C_0603_1608Metric -> Capacitor_SMD:C_0603_1608Metric_Pad1.08x0.95mm_HandSolder
- CP8, CP9: footprint Capacitor_Tantalum_SMD:CP_EIA-6032-28_Kemet-C -> Capacitor_Tantalum_SMD:CP_EIA-6032-28_Kemet-C_Pad2.25x2.35mm_HandSolder
- R11, R12, R13, R14, R6, R7: footprint Resistor_SMD:R_0603_1608Metric -> Resistor_SMD:R_0603_1608Metric_Pad0.98x0.95mm_HandSolder
Changed lines of the file:
@@
 F 0 "R11" H 1270 6446 50  0000 L CNN
 F 1 "100k" H 1270 6355 50  0000 L CNN
-F 2 "Resistor_SMD:R_0603_1608Metric" V 1130 6400 50  0001 C CNN
+F 2 "Resistor_SMD:R_0603_1608Metric_Pad0.98x0.95mm_HandSolder" V 1130 6400 50  0001 C CNN
 F 3 "~" H 1200 6400 50  0001 C CNN
 	1    1200 6400
@@
 F 0 "R12" H 1270 6846 50  0000 L CNN
 F 1 "100k" H 1270 6755 50  0000 L CNN
-F 2 "Resistor_SMD:R_0603_1608Metric" V 1130 6800 50  0001 C CNN
+F 2 "Resistor_SMD:R_0603_1608Metric_Pad0.98x0.95mm_HandSolder" V 1130 6800 50  0001 C CNN
 F 3 "~" H 1200 6800 50  0001 C CNN
 	1    1200 6800
@@
 F 0 "C6" H 3415 6496 50  0000 L CNN
 F 1 "47pF" H 3415 6405 50  0000 L CNN
-F 2 "Capacitor_SMD:C_0603_1608Metric" H 3338 6300 50  0001 C CNN
+F 2 "Capacitor_SMD:C_0603_1608Metric_Pad1.08x0.95mm_HandSolder" H 3338 6300 50  0001 C CNN
 F 3 "~" H 3300 6450 50  0001 C CNN
 	1    3300 6450
@@
 F 0 "R13" H 3820 6496 50  0000 L CNN
 F 1 "453k 1%" H 3820 6405 50  0000 L CNN
-F 2 "Resistor_SMD:R_0603_1608Metric" V 3680 6450 50  0001 C CNN
+F 2 "Resistor_SMD:R_0603_1608Metric_Pad0.98x0.95mm_HandSolder" V 3680 6450 50  0001 C CNN
 F 3 "~" H 3750 6450 50  0001 C CNN
 	1    3750 6450
@@
 F 0 "R14" H 3820 6946 50  0000 L CNN
 F 1 "100k 1%" H 3820 6855 50  0000 L CNN
-F 2 "Resistor_SMD:R_0603_1608Metric" V 3680 6900 50  0001 C CNN
+F 2 "Resistor_SMD:R_0603_1608Metric_Pad0.98x0.95mm_HandSolder" V 3680 6900 50  0001 C CNN
 F 3 "~" H 3750 6900 50  0001 C CNN
 	1    3750 6900
@@
 F 0 "CP8" H 4518 6496 50  0000 L CNN
 F 1 "22uF" H 4518 6405 50  0000 L CNN
-F 2 "Capacitor_Tantalum_SMD:CP_EIA-6032-28_Kemet-C" H 4438 6300 50  0001 C CNN
+F 2 "Capacitor_Tantalum_SMD:CP_EIA-6032-28_Kemet-C_Pad2.25x2.35mm_HandSolder" H 4438 6300 50  0001 C CNN
 F 3 "~" H 4400 6450 50  0001 C CNN
 	1    4400 6450
@@
 F 0 "CP9" H 5018 6496 50  0000 L CNN
 F 1 "22uF" H 5018 6405 50  0000 L CNN
-F 2 "Capacitor_Tantalum_SMD:CP_EIA-6032-28_Kemet-C" H 4938 6300 50  0001 C CNN
+F 2 "Capacitor_Tantalum_SMD:CP_EIA-6032-28_Kemet-C_Pad2.25x2.35mm_HandSolder" H 4938 6300 50  0001 C CNN
 F 3 "~" H 4900 6450 50  0001 C CNN
 	1    4900 6450
@@
 F 0 "R6" H 5620 1596 50  0000 L CNN
 F 1 "R" H 5620 1505 50  0000 L CNN
-F 2 "Resistor_SMD:R_0603_1608Metric" V 5480 1550 50  0001 C CNN
+F 2 "Resistor_SMD:R_0603_1608Metric_Pad0.98x0.95mm_HandSolder" V 5480 1550 50  0001 C CNN
 F 3 "~" H 5550 1550 50  0001 C CNN
 	1    5550 1550
@@
 F 0 "R7" H 5620 1996 50  0000 L CNN
 F 1 "R" H 5620 1905 50  0000 L CNN
-F 2 "Resistor_SMD:R_0603_1608Metric" V 5480 1950 50  0001 C CNN
+F 2 "Resistor_SMD:R_0603_1608Metric_Pad0.98x0.95mm_HandSolder" V 5480 1950 50  0001 C CNN
 F 3 "~" H 5550 1950 50  0001 C CNN
 	1    5550 1950
